Commit message: stl teste

File: config/arm.urdf (robot description, URDF)
Before this commit: robot test_robot, 8 links, 7 joints
Links:
- removed link base_cylinder
- removed link claw_base
- removed link claw_l
- removed link claw_r
- removed link lower_arm
- removed link platform
- removed link upper_arm
- removed link wrist
- added link 00; collision mesh filename=package://roboga_arm/meshes/00.stl scale=0.001 0.001 0.001; visual mesh filename=package://roboga_arm/meshes/00.stl scale=0.001 0.001 0.001
- added link 01; collision mesh filename=package://roboga_arm/meshes/01.stl; visual mesh filename=package://roboga_arm/meshes/01.stl
- added link 02; collision mesh filename=package://roboga_arm/meshes/02.stl; visual mesh filename=package://roboga_arm/meshes/02.stl
- added link 03; collision mesh filename=package://roboga_arm/meshes/03.stl; visual mesh filename=package://roboga_arm/meshes/03.stl
- added link 04; collision mesh filename=package://roboga_arm/meshes/04.stl; visual mesh filename=package://roboga_arm/meshes/04.stl
Joints:
- removed joint joint5
- removed joint joint6
- removed joint joint7
- joint joint1: child platform -> 01; parent base_cylinder -> 00
- joint joint2: child lower_arm -> 02; parent platform -> 01
- joint joint3: child upper_arm -> 03; parent lower_arm -> 02
- joint joint4: child wrist -> 04; parent upper_arm -> 03
